File: PCI_to_pinhead.kicad_sch (KiCad schematic)
At the start: 5 parts

Commit message: first attempt to order from PCBway
Parts:
- added H1, H2, H3, H4: MountingHole, MountingHole:MountingHole_3.2mm_M3, symbol Mechanical:MountingHole
- J1, J4: value (none) -> Conn_02x25_Odd_Even; footprint (none) -> Connector_PinHeader_2.54mm:PinHeader_2x25_P2.54mm_Vertical
- J2, J5: value (none) -> Conn_02x06_Odd_Even; footprint (none) -> Connector_PinHeader_2.54mm:PinHeader_2x06_P2.54mm_Vertical
- J3: value (none) -> Bus_PCI_32bit_5V; footprint (none) -> Connector_PCISlot:BUS_PCI_Slot
Changed lines of the file:
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@@
     (in_bom yes) (on_board yes)
     (property "Reference" "J3" (id 0) (at 95.25 16.0782 0))
-    (property "Value" "" (id 1) (at 95.25 18.3896 0))
-    (property "Footprint" "" (id 2) (at 95.25 100.33 0)
+    (property "Value" "Bus_PCI_32bit_5V" (id 1) (at 95.25 18.3896 0))
+    (property "Footprint" "Connector_PCISlot:BUS_PCI_Slot" (id 2) (at 95.25 100.33 0)
       (effects (font (size 1.27 1.27)) hide)
     )
@@
     (in_bom yes) (on_board yes)
     (property "Reference" "J1" (id 0) (at 36.83 32.5882 0))
-    (property "Value" "" (id 1) (at 36.83 34.8996 0))
-    (property "Footprint" "" (id 2) (at 35.56 68.58 0)
+    (property "Value" "Conn_02x25_Odd_Even" (id 1) (at 36.83 34.8996 0))
+    (property "Footprint" "Connector_PinHeader_2.54mm:PinHeader_2x25_P2.54mm_Vertical" (id 2) (at 35.56 68.58 0)
       (effects (font (size 1.27 1.27)) hide)
     )
@@
     (in_bom yes) (on_board yes)
     (property "Reference" "J2" (id 0) (at 36.83 146.8882 0))
-    (property "Value" "" (id 1) (at 36.83 149.1996 0))
-    (property "Footprint" "" (id 2) (at 35.56 157.48 0)
+    (property "Value" "Conn_02x06_Odd_Even" (id 1) (at 36.83 149.1996 0))
+    (property "Footprint" "Connector_PinHeader_2.54mm:PinHeader_2x06_P2.54mm_Vertical" (id 2) (at 35.56 157.48 0)
       (effects (font (size 1.27 1.27)) hide)
     )
@@
     (in_bom yes) (on_board yes)
     (property "Reference" "J5" (id 0) (at 154.94 146.8882 0))
-    (property "Value" "" (id 1) (at 154.94 149.1996 0))
-    (property "Footprint" "" (id 2) (at 153.67 157.48 0)
+    (property "Value" "Conn_02x06_Odd_Even" (id 1) (at 154.94 149.1996 0))
+    (property "Footprint" "Connector_PinHeader_2.54mm:PinHeader_2x06_P2.54mm_Vertical" (id 2) (at 153.67 157.48 0)
       (effects (font (size 1.27 1.27)) hide)
     )
@@
     (in_bom yes) (on_board yes)
     (property "Reference" "J4" (id 0) (at 154.94 32.5882 0))
-    (property "Value" "" (id 1) (at 154.94 34.8996 0))
-    (property "Footprint" "" (id 2) (at 153.67 68.58 0)
+    (property "Value" "Conn_02x25_Odd_Even" (id 1) (at 154.94 34.8996 0))
+    (property "Footprint" "Connector_PinHeader_2.54mm:PinHeader_2x25_P2.54mm_Vertical" (id 2) (at 153.67 68.58 0)
       (effects (font (size 1.27 1.27)) hide)
     )
@@
     (pin "9")
   )
+  (symbol (lib_id "Mechanical:MountingHole") (at 152.4 114.3 0) (unit 1)
+    (in_bom yes) (on_board yes) (fields_autoplaced)
+    (property "Reference" "H1" (id 0) (at 154.94 113.0299 0)
+      (effects (font (size 1.27 1.27)) (justify left))
+    )
+    (property "Value" "MountingHole" (id 1) (at 154.94 115.5699 0)
+      (effects (font (size 1.27 1.27)) (justify left))
+    )
+    (property "Footprint" "MountingHole:MountingHole_3.2mm_M3" (id 2) (at 152.4 114.3 0)
+      (effects (font (size 1.27 1.27)) hide)
+    )
+    (property "Datasheet" "~" (id 3) (at 152.4 114.3 0)
+      (effects (font (size 1.27 1.27)) hide)
+    )
+  )
+  (symbol (lib_id "Mechanical:MountingHole") (at 152.4 129.54 0) (unit 1)
+    (in_bom yes) (on_board yes) (fields_autoplaced)
+    (property "Reference" "H3" (id 0) (at 154.94 128.2699 0)
+      (effects (font (size 1.27 1.27)) (justify left))
+    )
+    (property "Value" "MountingHole" (id 1) (at 154.94 130.8099 0)
+      (effects (font (size 1.27 1.27)) (justify left))
+    )
+    (property "Footprint" "MountingHole:MountingHole_3.2mm_M3" (id 2) (at 152.4 129.54 0)
+      (effects (font (size 1.27 1.27)) hide)
+    )
+    (property "Datasheet" "~" (id 3) (at 152.4 129.54 0)
+      (effects (font (size 1.27 1.27)) hide)
+    )
+  )
+  (symbol (lib_id "Mechanical:MountingHole") (at 152.4 137.16 0) (unit 1)
+    (in_bom yes) (on_board yes) (fields_autoplaced)
+    (property "Reference" "H4" (id 0) (at 154.94 135.8899 0)
+      (effects (font (size 1.27 1.27)) (justify left))
+    )
+    (property "Value" "MountingHole" (id 1) (at 154.94 138.4299 0)
+      (effects (font (size 1.27 1.27)) (justify left))
+    )
+    (property "Footprint" "MountingHole:MountingHole_3.2mm_M3" (id 2) (at 152.4 137.16 0)
+      (effects (font (size 1.27 1.27)) hide)
+    )
+    (property "Datasheet" "~" (id 3) (at 152.4 137.16 0)
+      (effects (font (size 1.27 1.27)) hide)
+    )
+  )
+  (symbol (lib_id "Mechanical:MountingHole") (at 152.4 121.92 0) (unit 1)
+    (in_bom yes) (on_board yes) (fields_autoplaced)
+    (property "Reference" "H2" (id 0) (at 154.94 120.6499 0)
+      (effects (font (size 1.27 1.27)) (justify left))
+    )
+    (property "Value" "MountingHole" (id 1) (at 154.94 123.1899 0)
+      (effects (font (size 1.27 1.27)) (justify left))
+    )
+    (property "Footprint" "MountingHole:MountingHole_3.2mm_M3" (id 2) (at 152.4 121.92 0)
+      (effects (font (size 1.27 1.27)) hide)
+    )
+    (property "Datasheet" "~" (id 3) (at 152.4 121.92 0)
+      (effects (font (size 1.27 1.27)) hide)
+    )
+  )
   (sheet_instances
     (path "/" (page "1"))
   )
   (symbol_instances
+    (path "/620e855d-268a-460c-95b0-0fb81e740521"
+      (reference "H1") (unit 1) (value "MountingHole") (footprint "MountingHole:MountingHole_3.2mm_M3")
+    )
+    (path "/fb5af007-30b0-4d79-a224-7eefd42a8521"
+      (reference "H2") (unit 1) (value "MountingHole") (footprint "MountingHole:MountingHole_3.2mm_M3")
+    )
+    (path "/6d310e3d-bd53-4e6b-8e87-145a68a26811"
+      (reference "H3") (unit 1) (value "MountingHole") (footprint "MountingHole:MountingHole_3.2mm_M3")
+    )
+    (path "/8ce61696-ab02-4662-8341-66cd647973db"
+      (reference "H4") (unit 1) (value "MountingHole") (footprint "MountingHole:MountingHole_3.2mm_M3")
+    )
     (path "/00000000-0000-0000-0000-0000631b9128"
       (reference "J1") (unit 1) (value "Conn_02x25_Odd_Even") (footprint "Connector_PinHeader_2.54mm:PinHeader_2x25_P2.54mm_Vertical")
